Commit message: non-minimal example

File: resources/robots/mit_humanoid/urdf/humanoid_R_sf.urdf (robot description, URDF)
Before this commit: robot humanoid, 21 links, 20 joints
Joints:
- joint left_hip_abad: limit (none) -> lower=-6.28 upper=6.28 effort=34 velocity=50
- joint left_hip_yaw: limit (none) -> lower=-6.28 upper=6.28 effort=34 velocity=50

Commit message: this stays still

File: resources/robots/mit_humanoid/urdf/humanoid_R_sf.urdf (robot description, URDF)
Before this commit: robot humanoid, 21 links, 20 joints
Joints:
- joint left_ankle: type continuous -> revolute
- joint left_elbow: limit lower=-6.28 upper=6.28 effort=55 velocity=50 -> lower=-3 upper=3 effort=55 velocity=50; type continuous -> revolute
- joint left_hip_abad: limit lower=-6.28 upper=6.28 effort=34 velocity=50 -> lower=-3 upper=3 effort=34 velocity=50; type continuous -> revolute
- joint left_hip_pitch: limit lower=-6.28 upper=6.28 effort=72 velocity=50 -> lower=-3 upper=3 effort=72 velocity=50; type continuous -> revolute
- joint left_hip_yaw: limit lower=-6.28 upper=6.28 effort=34 velocity=50 -> lower=-3 upper=3 effort=34 velocity=50; type continuous -> revolute
- joint left_knee: type continuous -> revolute
- joint left_shoulder_abad: limit lower=-6.28 upper=6.28 effort=34 velocity=50 -> lower=-3 upper=3 effort=34 velocity=50; type continuous -> revolute
- joint left_shoulder_pitch: limit lower=-6.28 upper=6.28 effort=34 velocity=50 -> lower=-3 upper=3 effort=34 velocity=50; type continuous -> revolute
- joint left_shoulder_yaw: limit lower=-6.28 upper=6.28 effort=34 velocity=50 -> lower=-3 upper=3 effort=34 velocity=50; type continuous -> revolute
- joint right_ankle: type continuous -> revolute
- joint right_elbow: limit lower=-6.28 upper=6.28 effort=55 velocity=50 -> lower=-3 upper=3 effort=55 velocity=50; type continuous -> revolute
- joint right_hip_abad: limit lower=-6.28 upper=6.28 effort=34 velocity=50 -> lower=-3 upper=3 effort=34 velocity=50; type continuous -> revolute
- joint right_hip_pitch: limit lower=-6.28 upper=6.28 effort=72 velocity=50 -> lower=-3 upper=3 effort=72 velocity=50; type continuous -> revolute
- joint right_hip_yaw: limit lower=-6.28 upper=6.28 effort=34 velocity=50 -> lower=-3 upper=3 effort=34 velocity=50; type continuous -> revolute
- joint right_knee: type continuous -> revolute
- joint right_shoulder_abad: limit lower=-6.28 upper=6.28 effort=34 velocity=50 -> lower=-3 upper=3 effort=34 velocity=50; type continuous -> revolute
- joint right_shoulder_pitch: limit lower=-6.28 upper=6.28 effort=34 velocity=50 -> lower=-3 upper=3 effort=34 velocity=50; type continuous -> revolute
- joint right_shoulder_yaw: limit lower=-6.28 upper=6.28 effort=34 velocity=50 -> lower=-3 upper=3 effort=34 velocity=50; type continuous -> revolute

Commit message: disable motions

File: resources/robots/mit_humanoid/urdf/humanoid_R_sf.urdf (robot description, URDF)
Before this commit: robot humanoid, 21 links, 20 joints
Joints:
- joint left_ankle: type continuous -> revolute
- joint left_elbow: type continuous -> revolute
- joint left_hip_abad: type continuous -> revolute
- joint left_hip_pitch: type continuous -> revolute
- joint left_hip_yaw: type continuous -> revolute
- joint left_knee: type continuous -> revolute
- joint left_shoulder_abad: type continuous -> revolute
- joint left_shoulder_pitch: type continuous -> revolute
- joint left_shoulder_yaw: type continuous -> revolute
- joint right_ankle: type continuous -> revolute
- joint right_elbow: type continuous -> revolute
- joint right_hip_abad: type continuous -> revolute
- joint right_hip_pitch: type continuous -> revolute
- joint right_hip_yaw: type continuous -> revolute
- joint right_knee: type continuous -> revolute
- joint right_shoulder_abad: type continuous -> revolute
- joint right_shoulder_pitch: type continuous -> revolute
- joint right_shoulder_yaw: type continuous -> revolute
