Commit message: update all URDFs to work, add readme

File: resources/robots/mit_humanoid/urdf/humanoid_F_ht.urdf (robot description, URDF)
Before this commit: robot humanoid, 25 links, 24 joints
Joints:
- removed joint left_arm_pitch
- removed joint left_hip_abad_joint
- removed joint left_hip_yaw_joint
- removed joint right_arm_pitch
- removed joint right_hip_abad_joint
- removed joint right_hip_yaw_joint
- added joint left_hip_abad: type continuous, parent left_hip_yaw, child left_hip_abad, origin xyz=-0.06435 0 -.07499 rpy=0.0 0.436332 0.0, axis 1 0 0
- added joint left_hip_yaw: type continuous, parent base, child left_hip_yaw, origin xyz=0 0.082 0 rpy=0 -0.174533 0, axis 0 0 -1
- added joint left_shoulder_pitch: type continuous, parent base, child left_shoulder, origin xyz=0.01911 0.17608 0.30392 rpy=0 0 0, axis 0 1 0, limit lower=-6.28 upper=6.28 effort=34 velocity=50
- added joint right_hip_abad: type continuous, parent right_hip_yaw, child right_hip_abad, origin xyz=-0.06435 0 -.07499 rpy=0.0 0.436332 0.0, axis -1 0 0, limit lower=-6.28 upper=6.28 effort=34 velocity=50
- added joint right_hip_yaw: type continuous, parent base, child right_hip_yaw, origin xyz=0 -0.082 0 rpy=0 -0.174533 0, axis 0 0 1, limit lower=-6.28 upper=6.28 effort=34 velocity=50
- added joint right_shoulder_pitch: type continuous, parent base, child right_shoulder, origin xyz=0.01911 -0.17608 0.30392 rpy=0 0 0, axis 0 1 0, limit lower=-6.28 upper=6.28 effort=34 velocity=50

File: resources/robots/mit_humanoid/urdf/humanoid_R_ht.urdf (robot description, URDF)
Before this commit: robot humanoid, 25 links, 24 joints
Links:
- removed link leftlower
- removed link leftupper
- removed link rightlower
- removed link rightupper
- added link left_lower_leg, mass 0.346291; visual mesh filename=meshes_v3/left_leg_lower.stl scale=0.001 0.001 0.001
- added link left_upper_leg, mass 2.634789; visual mesh filename=meshes_v3/left_leg_upper.stl scale=0.001 0.001 0.001
- added link right_lower_leg, mass 0.346291; visual mesh filename=meshes_v3/left_leg_lower.stl scale=0.001 -0.001 0.001
- added link right_upper_leg, mass 2.634789; visual mesh filename=meshes_v3/left_leg_upper.stl scale=0.001 -0.001 0.001
- link base: geometry collision box size=0.15 0.3 0.35; visual mesh filename=meshes_v3/torso.stl scale=0.001 0.001 0.001
- link left_hand: geometry collision cylinder length=0.015 radius=0.025
- link right_hand: geometry collision cylinder length=0.015 radius=0.025
Joints:
- removed joint left_arm_pitch
- removed joint left_hip_abad_joint
- removed joint left_hip_yaw_joint
- removed joint right_arm_pitch
- removed joint right_hip_abad_joint
- removed joint right_hip_yaw_joint
- added joint left_hip_abad: type continuous, parent left_hip_yaw, child left_hip_abad, origin xyz=-0.06435 0 -.07499 rpy=0.0 0.436332 0.0, axis 1 0 0
- added joint left_hip_yaw: type continuous, parent base, child left_hip_yaw, origin xyz=0 0.082 0 rpy=0 -0.174533 0, axis 0 0 -1
- added joint left_shoulder_pitch: type continuous, parent base, child left_shoulder, origin xyz=0.01911 0.17608 0.30392 rpy=0 0 0, axis 0 1 0, limit lower=-6.28 upper=6.28 effort=34 velocity=50
- added joint right_hip_abad: type continuous, parent right_hip_yaw, child right_hip_abad, origin xyz=-0.06435 0 -.07499 rpy=0.0 0.436332 0.0, axis -1 0 0, limit lower=-6.28 upper=6.28 effort=34 velocity=50
- added joint right_hip_yaw: type continuous, parent base, child right_hip_yaw, origin xyz=0 -0.082 0 rpy=0 -0.174533 0, axis 0 0 1, limit lower=-6.28 upper=6.28 effort=34 velocity=50
- added joint right_shoulder_pitch: type continuous, parent base, child right_shoulder, origin xyz=0.01911 -0.17608 0.30392 rpy=0 0 0, axis 0 1 0, limit lower=-6.28 upper=6.28 effort=34 velocity=50
- joint left_ankle: parent leftlower -> left_lower_leg
- joint left_hip_pitch: child leftupper -> left_upper_leg
- joint left_knee: child leftlower -> left_lower_leg; parent leftupper -> left_upper_leg
- joint right_ankle: parent rightlower -> right_lower_leg
- joint right_hip_pitch: child rightupper -> right_upper_leg
- joint right_knee: child rightlower -> right_lower_leg; parent rightupper -> right_upper_leg

File: resources/robots/mit_humanoid/urdf/humanoid_R_sf.urdf (robot description, URDF)
Before this commit: robot humanoid, 21 links, 20 joints
Links:
- link left_hand: geometry collision cylinder length=0.015 radius=0.025
- link right_hand: geometry collision cylinder length=0.015 radius=0.025
Joints:
- removed joint ANKLE_L
- removed joint ANKLE_R
- removed joint ELBOW_L
- removed joint ELBOW_R
- removed joint HAND_L
- removed joint HAND_R
- removed joint HIP_aaL
- removed joint HIP_aaR
- removed joint HIP_pL
- removed joint HIP_pR
- removed joint HIP_yL
- removed joint HIP_yR
- removed joint KNEE_L
- removed joint KNEE_R
- removed joint SHOULDER_aaL
- removed joint SHOULDER_aaR
- removed joint SHOULDER_pL
- removed joint SHOULDER_pR
- removed joint SHOULDER_yL
- removed joint SHOULDER_yR
- added joint left_ankle: type continuous, parent left_lower_leg, child left_foot, origin xyz=0.0 0.0 -0.2785 rpy=0 0 0, axis 0 1 0, limit lower=-1.5 upper=1.5 effort=68 velocity=50
- added joint left_elbow: type continuous, parent left_upper_arm, child left_lower_arm, origin xyz=0 0 -.15750 rpy=0 0 0.0, axis 0 1 0, limit lower=-6.28 upper=6.28 effort=55 velocity=50
- added joint left_hand_link: type fixed, parent left_lower_arm, child left_hand, origin xyz=0 0 -0.27 rpy=0 0 0
- added joint left_hip_abad: type continuous, parent left_hip_yaw, child left_hip_abad, origin xyz=-0.06435 0 -.07499 rpy=0.0 0.436332 0.0, axis 1 0 0
- added joint left_hip_pitch: type continuous, parent left_hip_abad, child left_upper_leg, origin xyz=0.08837 -0.00284 -0.01385 rpy=0 -0.261799 0, axis 0 1 0, limit lower=-6.28 upper=6.28 effort=72 velocity=50
- added joint left_hip_yaw: type continuous, parent base, child left_hip_yaw, origin xyz=0 0.082 0 rpy=0 -0.174533 0, axis 0 0 -1
- added joint left_knee: type continuous, parent left_upper_leg, child left_lower_leg, origin xyz=-0.01306 0.0 -0.24916 rpy=0 0 0, axis 0 1 0, limit lower=0. upper=3. effort=144 velocity=50
- added joint left_shoulder_abad: type continuous, parent left_shoulder, child left_shoulder_2, origin xyz=0 .05760 0 rpy=0.0 0 0, axis 1 0 0, limit lower=-6.28 upper=6.28 effort=34 velocity=50
- added joint left_shoulder_pitch: type continuous, parent base, child left_shoulder, origin xyz=0.01911 0.17608 0.30392 rpy=0 0 0, axis 0 1 0, limit lower=-6.28 upper=6.28 effort=34 velocity=50
- added joint left_shoulder_yaw: type continuous, parent left_shoulder_2, child left_upper_arm, origin xyz=0 0 -.10250 rpy=0.0 0 0, axis 0 0 -1, limit lower=-6.28 upper=6.28 effort=34 velocity=50
- added joint right_ankle: type continuous, parent right_lower_leg, child right_foot, origin xyz=0.0 0.0 -0.2785 rpy=0 0 0, axis 0 1 0, limit lower=-1.5 upper=1.5 effort=68 velocity=50
- added joint right_elbow: type continuous, parent right_upper_arm, child right_lower_arm, origin xyz=0 0 -.15750 rpy=0 0 0.0, axis 0 1 0, limit lower=-6.28 upper=6.28 effort=55 velocity=50
- added joint right_hand_link: type fixed, parent right_lower_arm, child right_hand, origin xyz=0 0 -0.27 rpy=0 0 0
- added joint right_hip_abad: type continuous, parent right_hip_yaw, child right_hip_abad, origin xyz=-0.06435 0 -.07499 rpy=0.0 0.436332 0.0, axis -1 0 0, limit lower=-6.28 upper=6.28 effort=34 velocity=50
- added joint right_hip_pitch: type continuous, parent right_hip_abad, child right_upper_leg, origin xyz=0.08837 0.00284 -0.01385 rpy=0 -0.261799 0, axis 0 1 0, limit lower=-6.28 upper=6.28 effort=72 velocity=50
- added joint right_hip_yaw: type continuous, parent base, child right_hip_yaw, origin xyz=0 -0.082 0 rpy=0 -0.174533 0, axis 0 0 1, limit lower=-6.28 upper=6.28 effort=34 velocity=50
- added joint right_knee: type continuous, parent right_upper_leg, child right_lower_leg, origin xyz=-0.01306 0.0 -0.24916 rpy=0 0 0, axis 0 1 0, limit lower=0. upper=3.0 effort=144 velocity=50
- added joint right_shoulder_abad: type continuous, parent right_shoulder, child right_shoulder_2, origin xyz=0 -.05760 0 rpy=0.0 0 0, axis -1 0 0, limit lower=-6.28 upper=6.28 effort=34 velocity=50
- added joint right_shoulder_pitch: type continuous, parent base, child right_shoulder, origin xyz=0.01911 -0.17608 0.30392 rpy=0 0 0, axis 0 1 0, limit lower=-6.28 upper=6.28 effort=34 velocity=50
- added joint right_shoulder_yaw: type continuous, parent right_shoulder_2, child right_upper_arm, origin xyz=0 0 -.10250 rpy=0.0 0 0, axis 0 0 1, limit lower=-6.28 upper=6.28 effort=34 velocity=50

Commit message: fix all humanoid URDF collision bodies and joint types

File: resources/robots/mit_humanoid/urdf/humanoid_F_ht.urdf (robot description, URDF)
Before this commit: robot humanoid, 25 links, 24 joints
Joints:
- joint left_ankle: type continuous -> revolute
- joint left_elbow: type continuous -> revolute
- joint left_hip_abad: type continuous -> revolute
- joint left_hip_pitch: type continuous -> revolute
- joint left_hip_yaw: type continuous -> revolute
- joint left_knee: type continuous -> revolute
- joint left_shoulder_abad: type continuous -> revolute
- joint left_shoulder_pitch: type continuous -> revolute
- joint left_shoulder_yaw: type continuous -> revolute
- joint right_ankle: type continuous -> revolute
- joint right_elbow: type continuous -> revolute
- joint right_hip_abad: type continuous -> revolute
- joint right_hip_pitch: type continuous -> revolute
- joint right_hip_yaw: type continuous -> revolute
- joint right_knee: type continuous -> revolute
- joint right_shoulder_abad: type continuous -> revolute
- joint right_shoulder_pitch: type continuous -> revolute
- joint right_shoulder_yaw: type continuous -> revolute

File: resources/robots/mit_humanoid/urdf/humanoid_F_ht_b.urdf (robot description, URDF)
Before this commit: robot humanoid, 26 links, 25 joints
Joints:
- joint left_ankle: type continuous -> revolute
- joint left_elbow: type continuous -> revolute
- joint left_hip_abad: type continuous -> revolute
- joint left_hip_pitch: type continuous -> revolute
- joint left_hip_yaw: type continuous -> revolute
- joint left_knee: type continuous -> revolute
- joint left_shoulder_abad: type continuous -> revolute
- joint left_shoulder_pitch: type continuous -> revolute
- joint left_shoulder_yaw: type continuous -> revolute
- joint right_ankle: type continuous -> revolute
- joint right_elbow: type continuous -> revolute
- joint right_hip_abad: type continuous -> revolute
- joint right_hip_pitch: type continuous -> revolute
- joint right_hip_yaw: type continuous -> revolute
- joint right_knee: type continuous -> revolute
- joint right_shoulder_abad: type continuous -> revolute
- joint right_shoulder_pitch: type continuous -> revolute
- joint right_shoulder_yaw: type continuous -> revolute

File: resources/robots/mit_humanoid/urdf/humanoid_F_sf.urdf (robot description, URDF)
Before this commit: robot humanoid, 21 links, 20 joints
Joints:
- joint left_ankle: type continuous -> revolute
- joint left_elbow: type continuous -> revolute
- joint left_hip_abad: type continuous -> revolute
- joint left_hip_pitch: type continuous -> revolute
- joint left_hip_yaw: type continuous -> revolute
- joint left_knee: type continuous -> revolute
- joint left_shoulder_abad: type continuous -> revolute
- joint left_shoulder_pitch: type continuous -> revolute
- joint left_shoulder_yaw: type continuous -> revolute
- joint right_ankle: type continuous -> revolute
- joint right_elbow: type continuous -> revolute
- joint right_hip_abad: type continuous -> revolute
- joint right_hip_pitch: type continuous -> revolute
- joint right_hip_yaw: type continuous -> revolute
- joint right_knee: type continuous -> revolute
- joint right_shoulder_abad: type continuous -> revolute
- joint right_shoulder_pitch: type continuous -> revolute
- joint right_shoulder_yaw: type continuous -> revolute

File: resources/robots/mit_humanoid/urdf/humanoid_R_sf_b.urdf (robot description, URDF)
Before this commit: robot humanoid, 22 links, 21 joints
Links:
- link back: geometry collision mesh filename=meshes_v3/back.stl scale=0.001 0.001 0.001; visual mesh filename=meshes_v3/back.stl scale=0.001 0.001 0.001
- link base: geometry collision box size=0.15 0.3 0.35; visual mesh filename=meshes_v3/torso.stl scale=0.001 0.001 0.001

Commit message: Collapse joint fix (#13)
* initial commit, forked from dev

* debugging collapsing joints

* collapsed joint fixed. now contacts will register for fixed joints in urdf

* fixed other urdfs, adjusted default settings for humanoid

* fixed urdf with back geometry

File: resources/robots/mit_humanoid/urdf/humanoid_F_ht.urdf (robot description, URDF)
Before this commit: robot humanoid, 25 links, 24 joints
Links:
- link left_heel: mass 0.0 -> 0.001
- link left_toe: mass 0.0 -> 0.001
- link right_heel: mass 0.0 -> 0.001
- link right_toe: mass 0.0 -> 0.001
Joints:
- joint left_heel_link: origin xyz=0 -0.0 0 rpy=0 0 0 -> xyz=-0.05 0.0 -0.02 rpy=0 0 0
- joint left_toe_link: origin xyz=0 -0.0 0 rpy=0 0 0 -> xyz=0.085 0.0 -0.02 rpy=0 0 0
- joint right_heel_link: origin xyz=0 -0.0 0 rpy=0 0 0 -> xyz=0.085 0.0 -0.02 rpy=0 0 0
- joint right_toe_link: origin xyz=0 -0.0 0 rpy=0 0 0 -> xyz=0.085 0.0 -0.02 rpy=0 0 0

File: resources/robots/mit_humanoid/urdf/humanoid_R_ht.urdf (robot description, URDF)
Before this commit: robot humanoid, 25 links, 24 joints
Links:
- link left_hand: mass 0.0 -> 0.001
- link left_heel: mass 0.0 -> 0.001
- link left_toe: mass 0.0 -> 0.001
- link right_hand: mass 0.0 -> 0.001
- link right_heel: mass 0.0 -> 0.001
- link right_toe: mass 0.0 -> 0.001
Joints:
- joint left_elbow: limit lower=-6.28 upper=6.28 effort=55 velocity=50 -> lower=-3 upper=3 effort=55 velocity=50
- joint left_heel_link: origin xyz=0 -0.0 0 rpy=0 0 0 -> xyz=-0.05 0.0 -0.02 rpy=0 0 0
- joint left_hip_abad: limit (none) -> lower=-3 upper=3 effort=34 velocity=50
- joint left_hip_pitch: limit lower=-6.28 upper=6.28 effort=72 velocity=50 -> lower=-3 upper=3 effort=72 velocity=50
- joint left_hip_yaw: limit (none) -> lower=-3 upper=3 effort=34 velocity=50
- joint left_shoulder_abad: limit lower=-6.28 upper=6.28 effort=34 velocity=50 -> lower=-3 upper=3 effort=34 velocity=50
- joint left_shoulder_pitch: limit lower=-6.28 upper=6.28 effort=34 velocity=50 -> lower=-3 upper=3 effort=34 velocity=50
- joint left_shoulder_yaw: limit lower=-6.28 upper=6.28 effort=34 velocity=50 -> lower=-3 upper=3 effort=34 velocity=50
- joint left_toe_link: origin xyz=0 -0.0 0 rpy=0 0 0 -> xyz=0.085 0.0 -0.02 rpy=0 0 0
- joint right_elbow: limit lower=-6.28 upper=6.28 effort=55 velocity=50 -> lower=-3 upper=3 effort=55 velocity=50
- joint right_heel_link: origin xyz=0 -0.0 0 rpy=0 0 0 -> xyz=-0.05 0.0 -0.02 rpy=0 0 0
- joint right_hip_abad: limit lower=-6.28 upper=6.28 effort=34 velocity=50 -> lower=-3 upper=3 effort=34 velocity=50
- joint right_hip_pitch: limit lower=-6.28 upper=6.28 effort=72 velocity=50 -> lower=-3 upper=3 effort=72 velocity=50
- joint right_hip_yaw: limit lower=-6.28 upper=6.28 effort=34 velocity=50 -> lower=-3 upper=3 effort=34 velocity=50
- joint right_shoulder_abad: limit lower=-6.28 upper=6.28 effort=34 velocity=50 -> lower=-3 upper=3 effort=34 velocity=50
- joint right_shoulder_pitch: limit lower=-6.28 upper=6.28 effort=34 velocity=50 -> lower=-3 upper=3 effort=34 velocity=50
- joint right_shoulder_yaw: limit lower=-6.28 upper=6.28 effort=34 velocity=50 -> lower=-3 upper=3 effort=34 velocity=50
- joint right_toe_link: origin xyz=0 -0.0 0 rpy=0 0 0 -> xyz=0.085 0.0 -0.02 rpy=0 0 0
