Commit message: Humanoid URDF fixes (#123)
* update humanoid URDFs with numbering

* unifying humanoid URDFs, fixing several small bugs

* velocity limits updated

* one mistake

* collision meshes repaired

* unified URDFS

* make lower_legs match in length

---------

Co-authored-by: Elijah Stanger-Jones <elijahsj@mit.edu>

File: resources/robots/mit_humanoid/urdf/humanoid_F_ht.urdf (robot description, URDF)
Before this commit: robot humanoid, 25 links, 24 joints
Links:
- link left_hand: mass 0.0 -> 0.001
- link left_heel: geometry collision box size=0.06 0.04 0.02
- link left_toe: geometry collision box size=0.08 0.04 0.02
- link right_hand: mass 0.0 -> 0.001
- link right_heel: geometry collision box size=0.06 0.04 0.02
- link right_lower_leg: geometry collision cylinder length=0.16 radius=0.035; visual mesh filename=meshes_v3/left_leg_lower.stl scale=0.001 -0.001 0.001
- link right_toe: geometry collision box size=0.08 0.04 0.02
Joints:
- removed joint left_ankle
- removed joint left_elbow
- removed joint left_hip_abad
- removed joint left_hip_pitch
- removed joint left_hip_yaw
- removed joint left_knee
- removed joint left_shoulder_abad
- removed joint left_shoulder_pitch
- removed joint left_shoulder_yaw
- removed joint right_ankle
- removed joint right_elbow
- removed joint right_hip_abad
- removed joint right_hip_pitch
- removed joint right_hip_yaw
- removed joint right_knee
- removed joint right_shoulder_abad
- removed joint right_shoulder_pitch
- removed joint right_shoulder_yaw
- added joint 01_right_hip_yaw: type revolute, parent base, child right_hip_yaw, origin xyz=0 -0.082 0 rpy=0 -0.174533 0, axis 0 0 1, limit lower=-3 upper=3 effort=34 velocity=48
- added joint 02_right_hip_abad: type revolute, parent right_hip_yaw, child right_hip_abad, origin xyz=-0.06435 0 -.07499 rpy=0.0 0.436332 0.0, axis -1 0 0, limit lower=-3 upper=3 effort=34 velocity=48
- added joint 03_right_hip_pitch: type revolute, parent right_hip_abad, child right_upper_leg, origin xyz=0.08837 0.00284 -0.01385 rpy=0 -0.261799 0, axis 0 1 0, limit lower=-3 upper=3 effort=72 velocity=40
- added joint 04_right_knee: type revolute, parent right_upper_leg, child right_lower_leg, origin xyz=-0.01306 0.0 -0.24916 rpy=0 0 0, axis 0 1 0, limit lower=0. upper=3.0 effort=144 velocity=20
- added joint 05_right_ankle: type revolute, parent right_lower_leg, child right_foot, origin xyz=0.0 0.0 -0.2785 rpy=0 0 0, axis 0 1 0, limit lower=-1.5 upper=1.5 effort=68 velocity=24
- added joint 06_left_hip_yaw: type revolute, parent base, child left_hip_yaw, origin xyz=0 0.082 0 rpy=0 -0.174533 0, axis 0 0 -1, limit lower=-3 upper=3 effort=34 velocity=48
- added joint 07_left_hip_abad: type revolute, parent left_hip_yaw, child left_hip_abad, origin xyz=-0.06435 0 -.07499 rpy=0.0 0.436332 0.0, axis 1 0 0, limit lower=-3 upper=3 effort=34 velocity=48
- added joint 08_left_hip_pitch: type revolute, parent left_hip_abad, child left_upper_leg, origin xyz=0.08837 -0.00284 -0.01385 rpy=0 -0.261799 0, axis 0 1 0, limit lower=-3 upper=3 effort=72 velocity=40
- added joint 09_left_knee: type revolute, parent left_upper_leg, child left_lower_leg, origin xyz=-0.01306 0.0 -0.24916 rpy=0 0 0, axis 0 1 0, limit lower=0. upper=3. effort=144 velocity=20
- added joint 10_left_ankle: type revolute, parent left_lower_leg, child left_foot, origin xyz=0.0 0.0 -0.2785 rpy=0 0 0, axis 0 1 0, limit lower=-1.5 upper=1.5 effort=68 velocity=24
- added joint 11_right_shoulder_pitch: type revolute, parent base, child right_shoulder, origin xyz=0.01911 -0.17608 0.30392 rpy=0 0 0, axis 0 1 0, limit lower=-3 upper=3 effort=34 velocity=48
- added joint 12_right_shoulder_abad: type revolute, parent right_shoulder, child right_shoulder_2, origin xyz=0 -.05760 0 rpy=0.0 0 0, axis -1 0 0, limit lower=-3 upper=3 effort=34 velocity=48
- added joint 13_right_shoulder_yaw: type revolute, parent right_shoulder_2, child right_upper_arm, origin xyz=0 0 -.10250 rpy=0.0 0 0, axis 0 0 1, limit lower=-3 upper=3 effort=34 velocity=48
- added joint 14_right_elbow: type revolute, parent right_upper_arm, child right_lower_arm, origin xyz=0 0 -.15750 rpy=0 0 0.0, axis 0 1 0, limit lower=-3 upper=3 effort=55 velocity=30
- added joint 15_left_shoulder_pitch: type revolute, parent base, child left_shoulder, origin xyz=0.01911 0.17608 0.30392 rpy=0 0 0, axis 0 1 0, limit lower=-3 upper=3 effort=34 velocity=48
- added joint 16_left_shoulder_abad: type revolute, parent left_shoulder, child left_shoulder_2, origin xyz=0 .05760 0 rpy=0.0 0 0, axis 1 0 0, limit lower=-3 upper=3 effort=34 velocity=48
- added joint 17_left_shoulder_yaw: type revolute, parent left_shoulder_2, child left_upper_arm, origin xyz=0 0 -.10250 rpy=0.0 0 0, axis 0 0 -1, limit lower=-3 upper=3 effort=34 velocity=48
- added joint 18_left_elbow: type revolute, parent left_upper_arm, child left_lower_arm, origin xyz=0 0 -.15750 rpy=0 0 0.0, axis 0 1 0, limit lower=-3 upper=3 effort=55 velocity=30
- joint left_heel_link: origin xyz=-0.05 0.0 -0.02 rpy=0 0 0 -> xyz=-0.05 0.0 -0.03 rpy=0 0 0
- joint left_toe_link: origin xyz=0.085 0.0 -0.02 rpy=0 0 0 -> xyz=0.085 0.0 -0.03 rpy=0 0 0
- joint right_heel_link: origin xyz=0.085 0.0 -0.02 rpy=0 0 0 -> xyz=-0.05 0.0 -0.03 rpy=0 0 0
- joint right_toe_link: origin xyz=0.085 0.0 -0.02 rpy=0 0 0 -> xyz=0.085 0.0 -0.03 rpy=0 0 0

File: resources/robots/mit_humanoid/urdf/humanoid_F_ht_b.urdf (robot description, URDF)
Before this commit: robot humanoid, 26 links, 25 joints
Links:
- link left_hand: mass 0.0 -> 0.001
- link left_heel: mass 0.0 -> 0.001; geometry collision box size=0.06 0.04 0.02
- link left_toe: mass 0.0 -> 0.001; geometry collision box size=0.08 0.04 0.02
- link right_hand: mass 0.0 -> 0.001
- link right_heel: mass 0.0 -> 0.001; geometry collision box size=0.06 0.04 0.02
- link right_lower_leg: geometry collision cylinder length=0.16 radius=0.035; visual mesh filename=meshes_v3/left_leg_lower.stl scale=0.001 -0.001 0.001
- link right_toe: mass 0.0 -> 0.001; geometry collision box size=0.08 0.04 0.02
Joints:
- removed joint left_ankle
- removed joint left_elbow
- removed joint left_hip_abad
- removed joint left_hip_pitch
- removed joint left_hip_yaw
- removed joint left_knee
- removed joint left_shoulder_abad
- removed joint left_shoulder_pitch
- removed joint left_shoulder_yaw
- removed joint right_ankle
- removed joint right_elbow
- removed joint right_hip_abad
- removed joint right_hip_pitch
- removed joint right_hip_yaw
- removed joint right_knee
- removed joint right_shoulder_abad
- removed joint right_shoulder_pitch
- removed joint right_shoulder_yaw
- added joint 01_right_hip_yaw: type revolute, parent base, child right_hip_yaw, origin xyz=0 -0.082 0 rpy=0 -0.174533 0, axis 0 0 1, limit lower=-3 upper=3 effort=34 velocity=48
- added joint 02_right_hip_abad: type revolute, parent right_hip_yaw, child right_hip_abad, origin xyz=-0.06435 0 -.07499 rpy=0.0 0.436332 0.0, axis -1 0 0, limit lower=-3 upper=3 effort=34 velocity=48
- added joint 03_right_hip_pitch: type revolute, parent right_hip_abad, child right_upper_leg, origin xyz=0.08837 0.00284 -0.01385 rpy=0 -0.261799 0, axis 0 1 0, limit lower=-3 upper=3 effort=72 velocity=40
- added joint 04_right_knee: type revolute, parent right_upper_leg, child right_lower_leg, origin xyz=-0.01306 0.0 -0.24916 rpy=0 0 0, axis 0 1 0, limit lower=0. upper=3.0 effort=144 velocity=20
- added joint 05_right_ankle: type revolute, parent right_lower_leg, child right_foot, origin xyz=0.0 0.0 -0.2785 rpy=0 0 0, axis 0 1 0, limit lower=-1.5 upper=1.5 effort=68 velocity=24
- added joint 06_left_hip_yaw: type revolute, parent base, child left_hip_yaw, origin xyz=0 0.082 0 rpy=0 -0.174533 0, axis 0 0 -1, limit lower=-3 upper=3 effort=34 velocity=48
- added joint 07_left_hip_abad: type revolute, parent left_hip_yaw, child left_hip_abad, origin xyz=-0.06435 0 -.07499 rpy=0.0 0.436332 0.0, axis 1 0 0, limit lower=-3 upper=3 effort=34 velocity=48
- added joint 08_left_hip_pitch: type revolute, parent left_hip_abad, child left_upper_leg, origin xyz=0.08837 -0.00284 -0.01385 rpy=0 -0.261799 0, axis 0 1 0, limit lower=-3 upper=3 effort=72 velocity=40
- added joint 09_left_knee: type revolute, parent left_upper_leg, child left_lower_leg, origin xyz=-0.01306 0.0 -0.24916 rpy=0 0 0, axis 0 1 0, limit lower=0. upper=3. effort=144 velocity=20
- added joint 10_left_ankle: type revolute, parent left_lower_leg, child left_foot, origin xyz=0.0 0.0 -0.2785 rpy=0 0 0, axis 0 1 0, limit lower=-1.5 upper=1.5 effort=68 velocity=24
- added joint 11_right_shoulder_pitch: type revolute, parent base, child right_shoulder, origin xyz=0.01911 -0.17608 0.30392 rpy=0 0 0, axis 0 1 0, limit lower=-3 upper=3 effort=34 velocity=48
- added joint 12_right_shoulder_abad: type revolute, parent right_shoulder, child right_shoulder_2, origin xyz=0 -.05760 0 rpy=0.0 0 0, axis -1 0 0, limit lower=-3 upper=3 effort=34 velocity=48
- added joint 13_right_shoulder_yaw: type revolute, parent right_shoulder_2, child right_upper_arm, origin xyz=0 0 -.10250 rpy=0.0 0 0, axis 0 0 1, limit lower=-3 upper=3 effort=34 velocity=48
- added joint 14_right_elbow: type revolute, parent right_upper_arm, child right_lower_arm, origin xyz=0 0 -.15750 rpy=0 0 0.0, axis 0 1 0, limit lower=-3 upper=3 effort=55 velocity=30
- added joint 15_left_shoulder_pitch: type revolute, parent base, child left_shoulder, origin xyz=0.01911 0.17608 0.30392 rpy=0 0 0, axis 0 1 0, limit lower=-3 upper=3 effort=34 velocity=48
- added joint 16_left_shoulder_abad: type revolute, parent left_shoulder, child left_shoulder_2, origin xyz=0 .05760 0 rpy=0.0 0 0, axis 1 0 0, limit lower=-3 upper=3 effort=34 velocity=48
- added joint 17_left_shoulder_yaw: type revolute, parent left_shoulder_2, child left_upper_arm, origin xyz=0 0 -.10250 rpy=0.0 0 0, axis 0 0 -1, limit lower=-3 upper=3 effort=34 velocity=48
- added joint 18_left_elbow: type revolute, parent left_upper_arm, child left_lower_arm, origin xyz=0 0 -.15750 rpy=0 0 0.0, axis 0 1 0, limit lower=-3 upper=3 effort=55 velocity=30
- joint left_heel_link: origin xyz=0 -0.0 0 rpy=0 0 0 -> xyz=-0.05 0.0 -0.03 rpy=0 0 0
- joint left_toe_link: origin xyz=0 -0.0 0 rpy=0 0 0 -> xyz=0.085 0.0 -0.03 rpy=0 0 0
- joint right_heel_link: origin xyz=0 -0.0 0 rpy=0 0 0 -> xyz=-0.05 0.0 -0.03 rpy=0 0 0
- joint right_toe_link: origin xyz=0 -0.0 0 rpy=0 0 0 -> xyz=0.085 0.0 -0.03 rpy=0 0 0

File: resources/robots/mit_humanoid/urdf/humanoid_F_sf.urdf (robot description, URDF)
Before this commit: robot humanoid, 21 links, 20 joints
Links:
- link left_foot: geometry collision box size=0.20 0.02 0.04; visual mesh filename=meshes_v3/left_foot.stl scale=0.001 0.001 0.001
- link left_hand: mass 0.0 -> 0.001
- link right_foot: geometry collision box size=0.20 0.02 0.04; visual mesh filename=meshes_v3/left_foot.stl scale=0.001 -0.001 0.001
- link right_hand: mass 0.0 -> 0.001
- link right_lower_leg: geometry collision cylinder length=0.16 radius=0.035; visual mesh filename=meshes_v3/left_leg_lower.stl scale=0.001 -0.001 0.001
Joints:
- removed joint left_ankle
- removed joint left_elbow
- removed joint left_hip_abad
- removed joint left_hip_pitch
- removed joint left_hip_yaw
- removed joint left_knee
- removed joint left_shoulder_abad
- removed joint left_shoulder_pitch
- removed joint left_shoulder_yaw
- removed joint right_ankle
- removed joint right_elbow
- removed joint right_hip_abad
- removed joint right_hip_pitch
- removed joint right_hip_yaw
- removed joint right_knee
- removed joint right_shoulder_abad
- removed joint right_shoulder_pitch
- removed joint right_shoulder_yaw
- added joint 01_right_hip_yaw: type revolute, parent base, child right_hip_yaw, origin xyz=0 -0.082 0 rpy=0 -0.174533 0, axis 0 0 1, limit lower=-3 upper=3 effort=34 velocity=48
- added joint 02_right_hip_abad: type revolute, parent right_hip_yaw, child right_hip_abad, origin xyz=-0.06435 0 -.07499 rpy=0.0 0.436332 0.0, axis -1 0 0, limit lower=-3 upper=3 effort=34 velocity=48
- added joint 03_right_hip_pitch: type revolute, parent right_hip_abad, child right_upper_leg, origin xyz=0.08837 0.00284 -0.01385 rpy=0 -0.261799 0, axis 0 1 0, limit lower=-3 upper=3 effort=72 velocity=40
- added joint 04_right_knee: type revolute, parent right_upper_leg, child right_lower_leg, origin xyz=-0.01306 0.0 -0.24916 rpy=0 0 0, axis 0 1 0, limit lower=0. upper=3.0 effort=144 velocity=20
- added joint 05_right_ankle: type revolute, parent right_lower_leg, child right_foot, origin xyz=0.0 0.0 -0.2785 rpy=0 0 0, axis 0 1 0, limit lower=-1.5 upper=1.5 effort=68 velocity=24
- added joint 06_left_hip_yaw: type revolute, parent base, child left_hip_yaw, origin xyz=0 0.082 0 rpy=0 -0.174533 0, axis 0 0 -1, limit lower=-3 upper=3 effort=34 velocity=48
- added joint 07_left_hip_abad: type revolute, parent left_hip_yaw, child left_hip_abad, origin xyz=-0.06435 0 -.07499 rpy=0.0 0.436332 0.0, axis 1 0 0, limit lower=-3 upper=3 effort=34 velocity=48
- added joint 08_left_hip_pitch: type revolute, parent left_hip_abad, child left_upper_leg, origin xyz=0.08837 -0.00284 -0.01385 rpy=0 -0.261799 0, axis 0 1 0, limit lower=-3 upper=3 effort=72 velocity=40
- added joint 09_left_knee: type revolute, parent left_upper_leg, child left_lower_leg, origin xyz=-0.01306 0.0 -0.24916 rpy=0 0 0, axis 0 1 0, limit lower=0. upper=3. effort=144 velocity=20
- added joint 10_left_ankle: type revolute, parent left_lower_leg, child left_foot, origin xyz=0.0 0.0 -0.2785 rpy=0 0 0, axis 0 1 0, limit lower=-1.5 upper=1.5 effort=68 velocity=24
- added joint 11_right_shoulder_pitch: type revolute, parent base, child right_shoulder, origin xyz=0.01911 -0.17608 0.30392 rpy=0 0 0, axis 0 1 0, limit lower=-3 upper=3 effort=34 velocity=48
- added joint 12_right_shoulder_abad: type revolute, parent right_shoulder, child right_shoulder_2, origin xyz=0 -.05760 0 rpy=0.0 0 0, axis -1 0 0, limit lower=-3 upper=3 effort=34 velocity=48
- added joint 13_right_shoulder_yaw: type revolute, parent right_shoulder_2, child right_upper_arm, origin xyz=0 0 -.10250 rpy=0.0 0 0, axis 0 0 1, limit lower=-3 upper=3 effort=34 velocity=48
- added joint 14_right_elbow: type revolute, parent right_upper_arm, child right_lower_arm, origin xyz=0 0 -.15750 rpy=0 0 0.0, axis 0 1 0, limit lower=-3 upper=3 effort=55 velocity=30
- added joint 15_left_shoulder_pitch: type revolute, parent base, child left_shoulder, origin xyz=0.01911 0.17608 0.30392 rpy=0 0 0, axis 0 1 0, limit lower=-3 upper=3 effort=34 velocity=48
- added joint 16_left_shoulder_abad: type revolute, parent left_shoulder, child left_shoulder_2, origin xyz=0 .05760 0 rpy=0.0 0 0, axis 1 0 0, limit lower=-3 upper=3 effort=34 velocity=48
- added joint 17_left_shoulder_yaw: type revolute, parent left_shoulder_2, child left_upper_arm, origin xyz=0 0 -.10250 rpy=0.0 0 0, axis 0 0 -1, limit lower=-3 upper=3 effort=34 velocity=48
- added joint 18_left_elbow: type revolute, parent left_upper_arm, child left_lower_arm, origin xyz=0 0 -.15750 rpy=0 0 0.0, axis 0 1 0, limit lower=-3 upper=3 effort=55 velocity=30

File: resources/robots/mit_humanoid/urdf/humanoid_R_ht.urdf (robot description, URDF)
Before this commit: robot humanoid, 25 links, 24 joints
Links:
- link left_heel: geometry collision box size=0.06 0.04 0.02
- link left_toe: geometry collision box size=0.08 0.04 0.02
- link right_heel: geometry collision box size=0.06 0.04 0.02
- link right_toe: geometry collision box size=0.08 0.04 0.02
Joints:
- removed joint left_elbow
- removed joint left_hip_abad
- removed joint left_hip_pitch
- removed joint left_hip_yaw
- removed joint left_knee
- removed joint left_shoulder_abad
- removed joint left_shoulder_pitch
- removed joint left_shoulder_yaw
- removed joint right_ankle
- removed joint right_elbow
- removed joint right_hip_abad
- removed joint right_hip_pitch
- removed joint right_hip_yaw
- removed joint right_knee
- removed joint right_shoulder_abad
- removed joint right_shoulder_pitch
- removed joint right_shoulder_yaw
- added joint 01_right_hip_yaw: type revolute, parent base, child right_hip_yaw, origin xyz=0 -0.082 0 rpy=0 -0.174533 0, axis 0 0 1, limit lower=-3 upper=3 effort=34 velocity=48
- added joint 02_right_hip_abad: type revolute, parent right_hip_yaw, child right_hip_abad, origin xyz=-0.06435 0 -.07499 rpy=0.0 0.436332 0.0, axis -1 0 0, limit lower=-3 upper=3 effort=34 velocity=48
- added joint 03_right_hip_pitch: type revolute, parent right_hip_abad, child right_upper_leg, origin xyz=0.08837 0.00284 -0.01385 rpy=0 -0.261799 0, axis 0 1 0, limit lower=-3 upper=3 effort=72 velocity=40
- added joint 04_right_knee: type revolute, parent right_upper_leg, child right_lower_leg, origin xyz=-0.01306 0.0 -0.24916 rpy=0 0 0, axis 0 1 0, limit lower=0. upper=3.0 effort=144 velocity=20
- added joint 05_right_ankle: type revolute, parent right_lower_leg, child right_foot, origin xyz=0.0 0.0 -0.2785 rpy=0 0 0, axis 0 1 0, limit lower=-1.5 upper=1.5 effort=68 velocity=24
- added joint 06_left_hip_yaw: type revolute, parent base, child left_hip_yaw, origin xyz=0 0.082 0 rpy=0 -0.174533 0, axis 0 0 -1, limit lower=-3 upper=3 effort=34 velocity=48
- added joint 07_left_hip_abad: type revolute, parent left_hip_yaw, child left_hip_abad, origin xyz=-0.06435 0 -.07499 rpy=0.0 0.436332 0.0, axis 1 0 0, limit lower=-3 upper=3 effort=34 velocity=48
- added joint 08_left_hip_pitch: type revolute, parent left_hip_abad, child left_upper_leg, origin xyz=0.08837 -0.00284 -0.01385 rpy=0 -0.261799 0, axis 0 1 0, limit lower=-3 upper=3 effort=72 velocity=40
- added joint 09_left_knee: type revolute, parent left_upper_leg, child left_lower_leg, origin xyz=-0.01306 0.0 -0.24916 rpy=0 0 0, axis 0 1 0, limit lower=0. upper=3. effort=144 velocity=20
- added joint 11_right_shoulder_pitch: type revolute, parent base, child right_shoulder, origin xyz=0.01911 -0.17608 0.30392 rpy=0 0 0, axis 0 1 0, limit lower=-3 upper=3 effort=34 velocity=48
- added joint 12_right_shoulder_abad: type revolute, parent right_shoulder, child right_shoulder_2, origin xyz=0 -.05760 0 rpy=0.0 0 0, axis -1 0 0, limit lower=-3 upper=3 effort=34 velocity=48
- added joint 13_right_shoulder_yaw: type revolute, parent right_shoulder_2, child right_upper_arm, origin xyz=0 0 -.10250 rpy=0.0 0 0, axis 0 0 1, limit lower=-3 upper=3 effort=34 velocity=48
- added joint 14_right_elbow: type revolute, parent right_upper_arm, child right_lower_arm, origin xyz=0 0 -.15750 rpy=0 0 0.0, axis 0 1 0, limit lower=-3 upper=3 effort=55 velocity=30
- added joint 15_left_shoulder_pitch: type revolute, parent base, child left_shoulder, origin xyz=0.01911 0.17608 0.30392 rpy=0 0 0, axis 0 1 0, limit lower=-3 upper=3 effort=34 velocity=48
- added joint 16_left_shoulder_abad: type revolute, parent left_shoulder, child left_shoulder_2, origin xyz=0 .05760 0 rpy=0.0 0 0, axis 1 0 0, limit lower=-3 upper=3 effort=34 velocity=48
- added joint 17_left_shoulder_yaw: type revolute, parent left_shoulder_2, child left_upper_arm, origin xyz=0 0 -.10250 rpy=0.0 0 0, axis 0 0 -1, limit lower=-3 upper=3 effort=34 velocity=48
- added joint 18_left_elbow: type revolute, parent left_upper_arm, child left_lower_arm, origin xyz=0 0 -.15750 rpy=0 0 0.0, axis 0 1 0, limit lower=-3 upper=3 effort=55 velocity=30
- joint left_ankle: limit lower=-1.5 upper=1.5 effort=68 velocity=50 -> lower=-1.5 upper=1.5 effort=68 velocity=24
- joint left_heel_link: origin xyz=-0.05 0.0 -0.02 rpy=0 0 0 -> xyz=-0.05 0.0 -0.03 rpy=0 0 0
- joint left_toe_link: origin xyz=0.085 0.0 -0.02 rpy=0 0 0 -> xyz=0.085 0.0 -0.03 rpy=0 0 0
- joint right_heel_link: origin xyz=-0.05 0.0 -0.02 rpy=0 0 0 -> xyz=-0.05 0.0 -0.03 rpy=0 0 0
- joint right_toe_link: origin xyz=0.085 0.0 -0.02 rpy=0 0 0 -> xyz=0.085 0.0 -0.03 rpy=0 0 0
