Commit message: minor edits in the urdf

File: resources/robots/mini_cheetah/urdf/mini_cheetah.urdf (robot description, URDF)
Before this commit: robot mini_cheetah_vision, 13 links, 12 joints
Links:
- removed link abduct_fl
- removed link abduct_fr
- removed link abduct_hl
- removed link abduct_hr
- removed link body
- removed link shank_fl
- removed link shank_fr
- removed link shank_hl
- removed link shank_hr
- removed link thigh_fl
- removed link thigh_fr
- removed link thigh_hl
- removed link thigh_hr
- added link LF_FOOT, mass 0.01; collision sphere radius=0.031
- added link LF_HIP, mass 0.54; collision mesh filename=meshes/mini_vision_abd.dae; visual mesh filename=meshes/mini_vision_abd.dae
- added link LF_SHANK, mass 0.064; collision mesh filename=meshes/lower_leg.dae; visual mesh filename=meshes/lower_leg.dae
- added link LF_THIGH, mass 0.634; collision mesh filename=meshes/mini_vision_upper_leg.dae; visual mesh filename=meshes/mini_vision_upper_leg.dae
- added link LH_FOOT, mass 0.01; collision sphere radius=0.031
- added link LH_HIP, mass 0.54; collision mesh filename=meshes/mini_vision_abd.dae; visual mesh filename=meshes/mini_vision_abd.dae
- added link LH_SHANK, mass 0.064; collision mesh filename=meshes/lower_leg.dae; visual mesh filename=meshes/lower_leg.dae
- added link LH_THIGH, mass 0.634; collision mesh filename=meshes/mini_vision_upper_leg.dae; visual mesh filename=meshes/mini_vision_upper_leg.dae
- added link RF_FOOT, mass 0.01; collision sphere radius=0.031
- added link RF_HIP, mass 0.54; collision mesh filename=meshes/mini_vision_abd.dae; visual mesh filename=meshes/mini_vision_abd.dae
- added link RF_SHANK, mass 0.064; collision mesh filename=meshes/lower_leg.dae; visual mesh filename=meshes/lower_leg.dae
- added link RF_THIGH, mass 0.634; collision mesh filename=meshes/mini_vision_upper_leg.dae; visual mesh filename=meshes/mini_vision_upper_leg.dae
- added link RH_FOOT, mass 0.01; collision sphere radius=0.031
- added link RH_HIP, mass 0.54; collision mesh filename=meshes/mini_vision_abd.dae; visual mesh filename=meshes/mini_vision_abd.dae
- added link RH_SHANK, mass 0.064; collision mesh filename=meshes/lower_leg.dae; visual mesh filename=meshes/lower_leg.dae
- added link RH_THIGH, mass 0.634; collision mesh filename=meshes/mini_vision_upper_leg.dae; visual mesh filename=meshes/mini_vision_upper_leg.dae
- added link base, mass 3.3; collision mesh filename=meshes/mini_vision_body.dae; visual mesh filename=meshes/mini_vision_body.dae
Joints:
- removed joint abduct_fl_to_thigh_fl_j
- removed joint abduct_fr_to_thigh_fr_j
- removed joint abduct_hl_to_thigh_hl_j
- removed joint abduct_hr_to_thigh_hr_j
- removed joint thigh_fl_to_knee_fl_j
- removed joint thigh_fr_to_knee_fr_j
- removed joint thigh_hl_to_knee_hl_j
- removed joint thigh_hr_to_knee_hr_j
- removed joint torso_to_abduct_fl_j
- removed joint torso_to_abduct_fr_j
- removed joint torso_to_abduct_hl_j
- removed joint torso_to_abduct_hr_j
- added joint LF_HAA: type revolute, parent base, child LF_HIP, origin xyz=0.14775 0.049 0.0 rpy=0 0 0, axis 1 0 0, limit lower=-6.28 upper=6.28 effort=72 velocity=50
- added joint LF_HFE: type revolute, parent LF_HIP, child LF_THIGH, origin xyz=0.055 0.019 0.00 rpy=0.0 0.0 0.0, axis 0 -1 0, limit lower=-6.28 upper=6.28 effort=72 velocity=50
- added joint LF_KFE: type revolute, parent LF_THIGH, child LF_SHANK, origin xyz=0.0 0.049 -0.2085 rpy=0.0 0 0.0, axis 0 -1 0, limit lower=-6.28 upper=6.28 effort=72 velocity=50
- added joint LF_SHANK_TO_FOOT: type fixed, parent LF_SHANK, child LF_FOOT, origin xyz=0.0 0.0 -0.32125 rpy=0.0 0.0 0.0
- added joint LH_HAA: type revolute, parent base, child LH_HIP, origin xyz=-0.14775 0.049 0.0 rpy=0 3.141592 0, axis -1 0 0, limit lower=-6.28 upper=6.28 effort=72 velocity=50
- added joint LH_HFE: type revolute, parent LH_HIP, child LH_THIGH, origin xyz=0.055 0.019 0.00 rpy=0.0 3.141592 0.0, axis 0 -1 0, limit lower=-6.28 upper=6.28 effort=72 velocity=50
- added joint LH_KFE: type revolute, parent LH_THIGH, child LH_SHANK, origin xyz=0.0 0.049 -0.2085 rpy=0.0 0 0.0, axis 0 -1 0, limit lower=-6.28 upper=6.28 effort=72 velocity=50
- added joint LH_SHANK_TO_FOOT: type fixed, parent LH_SHANK, child LH_FOOT, origin xyz=0.0 0.0 -0.32125 rpy=0.0 0.0 0.0
- added joint RF_HAA: type revolute, parent base, child RF_HIP, origin xyz=0.14775 -0.049 0.0 rpy=0 0 0, axis 1 0 0, limit lower=-6.28 upper=6.28 effort=72 velocity=50
- added joint RF_HFE: type revolute, parent RF_HIP, child RF_THIGH, origin xyz=0.055 -0.019 0.00 rpy=0.0 0.0 0.0, axis 0 -1 0, limit lower=-6.28 upper=6.28 effort=72 velocity=50
- added joint RF_KFE: type revolute, parent RF_THIGH, child RF_SHANK, origin xyz=0.0 -0.049 -0.2085 rpy=0.0 0 0.0, axis 0 -1 0, limit lower=-6.28 upper=6.28 effort=72 velocity=50
- added joint RF_SHANK_TO_FOOT: type fixed, parent RF_SHANK, child RF_FOOT, origin xyz=0.0 0.0 -0.32125 rpy=0.0 0.0 0.0
- added joint RH_HAA: type revolute, parent base, child RH_HIP, origin xyz=-0.14775 -0.049 0.0 rpy=0 3.141592 0, axis -1 0 0, limit lower=-6.28 upper=6.28 effort=72 velocity=50
- added joint RH_HFE: type revolute, parent RH_HIP, child RH_THIGH, origin xyz=0.055 -0.019 0.00 rpy=0.0 3.141592 0.0, axis 0 -1 0, limit lower=-6.28 upper=6.28 effort=72 velocity=50
- added joint RH_KFE: type revolute, parent RH_THIGH, child RH_SHANK, origin xyz=0.0 -0.049 -0.2085 rpy=0.0 0 0.0, axis 0 -1 0, limit lower=-6.28 upper=6.28 effort=72 velocity=50
- added joint RH_SHANK_TO_FOOT: type fixed, parent RH_SHANK, child RH_FOOT, origin xyz=0.0 0.0 -0.32125 rpy=0.0 0.0 0.0

Commit message: adding new joint limits and fixing the foot contact with the minicheetah urdf

File: resources/robots/mini_cheetah/urdf/mini_cheetah.urdf (robot description, URDF)
Before this commit: robot mini_cheetah_vision, 17 links, 16 joints
Links:
- link LF_FOOT: geometry collision sphere radius=0.02
- link LH_FOOT: geometry collision sphere radius=0.02
- link RF_FOOT: geometry collision sphere radius=0.02
- link RH_FOOT: geometry collision sphere radius=0.02
Joints:
- joint LF_HAA: limit lower=-6.28 upper=6.28 effort=72 velocity=50 -> lower=-1.6 upper=1.6 effort=18 velocity=40
- joint LF_HFE: limit lower=-6.28 upper=6.28 effort=72 velocity=50 -> lower=-2.6 upper=2.6 effort=18 velocity=40
- joint LF_KFE: limit lower=-6.28 upper=6.28 effort=72 velocity=50 -> lower=-2.6 upper=2.6 effort=26 velocity=26
- joint LF_SHANK_TO_FOOT: origin xyz=0.0 0.0 -0.32125 rpy=0.0 0.0 0.0 -> xyz=0.0 0.0 -0.22 rpy=0.0 0.0 0.0
- joint LH_HAA: limit lower=-6.28 upper=6.28 effort=72 velocity=50 -> lower=-1.6 upper=1.6 effort=18 velocity=40
- joint LH_HFE: limit lower=-6.28 upper=6.28 effort=72 velocity=50 -> lower=-2.6 upper=2.6 effort=18 velocity=40
- joint LH_KFE: limit lower=-6.28 upper=6.28 effort=72 velocity=50 -> lower=-2.6 upper=2.6 effort=18 velocity=40
- joint LH_SHANK_TO_FOOT: origin xyz=0.0 0.0 -0.32125 rpy=0.0 0.0 0.0 -> xyz=0.0 0.0 -0.22 rpy=0.0 0.0 0.0
- joint RF_HAA: limit lower=-6.28 upper=6.28 effort=72 velocity=50 -> lower=-1.6 upper=1.6 effort=18 velocity=40
- joint RF_HFE: limit lower=-6.28 upper=6.28 effort=72 velocity=50 -> lower=-2.6 upper=2.6 effort=18 velocity=40
- joint RF_KFE: limit lower=-6.28 upper=6.28 effort=72 velocity=50 -> lower=-2.6 upper=2.6 effort=18 velocity=40
- joint RF_SHANK_TO_FOOT: origin xyz=0.0 0.0 -0.32125 rpy=0.0 0.0 0.0 -> xyz=0.0 0.0 -0.22 rpy=0.0 0.0 0.0
- joint RH_HAA: limit lower=-6.28 upper=6.28 effort=72 velocity=50 -> lower=-1.6 upper=1.6 effort=18 velocity=40
- joint RH_HFE: limit lower=-6.28 upper=6.28 effort=72 velocity=50 -> lower=-2.6 upper=2.6 effort=18 velocity=40
- joint RH_KFE: limit lower=-6.28 upper=6.28 effort=72 velocity=50 -> lower=-2.6 upper=2.6 effort=18 velocity=40
- joint RH_SHANK_TO_FOOT: origin xyz=0.0 0.0 -0.32125 rpy=0.0 0.0 0.0 -> xyz=0.0 0.0 -0.22 rpy=0.0 0.0 0.0

Commit message: cosmetic changes mini cheetah urdf

File: resources/robots/mini_cheetah/urdf/mini_cheetah.urdf (robot description, URDF)
Before this commit: robot mini_cheetah_vision, 17 links, 16 joints
Links:
- removed link LF_FOOT
- removed link LF_HIP
- removed link LF_SHANK
- removed link LF_THIGH
- removed link LH_FOOT
- removed link LH_HIP
- removed link LH_SHANK
- removed link LH_THIGH
- removed link RF_FOOT
- removed link RF_HIP
- removed link RF_SHANK
- removed link RF_THIGH
- removed link RH_FOOT
- removed link RH_HIP
- removed link RH_SHANK
- removed link RH_THIGH
- added link lf_foot, mass 0.01; collision sphere radius=0.02
- added link lf_hip, mass 0.54; collision mesh filename=meshes/mini_vision_abd.dae; visual mesh filename=meshes/mini_vision_abd.dae
- added link lf_shank, mass 0.064; collision mesh filename=meshes/lower_leg.dae; visual mesh filename=meshes/lower_leg.dae
- added link lf_thigh, mass 0.634; collision mesh filename=meshes/mini_vision_upper_leg.dae; visual mesh filename=meshes/mini_vision_upper_leg.dae
- added link lh_foot, mass 0.01; collision sphere radius=0.02
- added link lh_hip, mass 0.54; collision mesh filename=meshes/mini_vision_abd.dae; visual mesh filename=meshes/mini_vision_abd.dae
- added link lh_shank, mass 0.064; collision mesh filename=meshes/lower_leg.dae; visual mesh filename=meshes/lower_leg.dae
- added link lh_thigh, mass 0.634; collision mesh filename=meshes/mini_vision_upper_leg.dae; visual mesh filename=meshes/mini_vision_upper_leg.dae
- added link rf_foot, mass 0.01; collision sphere radius=0.02
- added link rf_hip, mass 0.54; collision mesh filename=meshes/mini_vision_abd.dae; visual mesh filename=meshes/mini_vision_abd.dae
- added link rf_shank, mass 0.064; collision mesh filename=meshes/lower_leg.dae; visual mesh filename=meshes/lower_leg.dae
- added link rf_thigh, mass 0.634; collision mesh filename=meshes/mini_vision_upper_leg.dae; visual mesh filename=meshes/mini_vision_upper_leg.dae
- added link rh_foot, mass 0.01; collision sphere radius=0.02
- added link rh_hip, mass 0.54; collision mesh filename=meshes/mini_vision_abd.dae; visual mesh filename=meshes/mini_vision_abd.dae
- added link rh_shank, mass 0.064; collision mesh filename=meshes/lower_leg.dae; visual mesh filename=meshes/lower_leg.dae
- added link rh_thigh, mass 0.634; collision mesh filename=meshes/mini_vision_upper_leg.dae; visual mesh filename=meshes/mini_vision_upper_leg.dae
Joints:
- removed joint LF_HAA
- removed joint LF_HFE
- removed joint LF_KFE
- removed joint LF_SHANK_TO_FOOT
- removed joint LH_HAA
- removed joint LH_HFE
- removed joint LH_KFE
- removed joint LH_SHANK_TO_FOOT
- removed joint RF_HAA
- removed joint RF_HFE
- removed joint RF_KFE
- removed joint RF_SHANK_TO_FOOT
- removed joint RH_HAA
- removed joint RH_HFE
- removed joint RH_KFE
- removed joint RH_SHANK_TO_FOOT
- added joint lf_haa: type revolute, parent base, child lf_hip, origin xyz=0.14775 0.049 0.0 rpy=0 0 0, axis 1 0 0, limit lower=-1.6 upper=1.6 effort=18 velocity=40
- added joint lf_hfe: type revolute, parent lf_hip, child lf_thigh, origin xyz=0.055 0.019 0.00 rpy=0.0 0.0 0.0, axis 0 -1 0, limit lower=-2.6 upper=2.6 effort=18 velocity=40
- added joint lf_kfe: type revolute, parent lf_thigh, child lf_shank, origin xyz=0.0 0.049 -0.2085 rpy=0.0 0 0.0, axis 0 -1 0, limit lower=-2.6 upper=2.6 effort=26 velocity=26
- added joint lf_shank_to_foot: type fixed, parent lf_shank, child lf_foot, origin xyz=0.0 0.0 -0.22 rpy=0.0 0.0 0.0
- added joint lh_haa: type revolute, parent base, child lh_hip, origin xyz=-0.14775 0.049 0.0 rpy=0 3.141592 0, axis -1 0 0, limit lower=-1.6 upper=1.6 effort=18 velocity=40
- added joint lh_hfe: type revolute, parent lh_hip, child lh_thigh, origin xyz=0.055 0.019 0.00 rpy=0.0 3.141592 0.0, axis 0 -1 0, limit lower=-2.6 upper=2.6 effort=18 velocity=40
- added joint lh_kfe: type revolute, parent lh_thigh, child lh_shank, origin xyz=0.0 0.049 -0.2085 rpy=0.0 0 0.0, axis 0 -1 0, limit lower=-2.6 upper=2.6 effort=18 velocity=40
- added joint lh_shank_to_foot: type fixed, parent lh_shank, child lh_foot, origin xyz=0.0 0.0 -0.22 rpy=0.0 0.0 0.0
- added joint rf_haa: type revolute, parent base, child rf_hip, origin xyz=0.14775 -0.049 0.0 rpy=0 0 0, axis 1 0 0, limit lower=-1.6 upper=1.6 effort=18 velocity=40
- added joint rf_hfe: type revolute, parent rf_hip, child rf_thigh, origin xyz=0.055 -0.019 0.00 rpy=0.0 0.0 0.0, axis 0 -1 0, limit lower=-2.6 upper=2.6 effort=18 velocity=40
- added joint rf_kfe: type revolute, parent rf_thigh, child rf_shank, origin xyz=0.0 -0.049 -0.2085 rpy=0.0 0 0.0, axis 0 -1 0, limit lower=-2.6 upper=2.6 effort=18 velocity=40
- added joint rf_shank_to_foot: type fixed, parent rf_shank, child rf_foot, origin xyz=0.0 0.0 -0.22 rpy=0.0 0.0 0.0
- added joint rh_haa: type revolute, parent base, child rh_hip, origin xyz=-0.14775 -0.049 0.0 rpy=0 3.141592 0, axis -1 0 0, limit lower=-1.6 upper=1.6 effort=18 velocity=40
- added joint rh_hfe: type revolute, parent rh_hip, child rh_thigh, origin xyz=0.055 -0.019 0.00 rpy=0.0 3.141592 0.0, axis 0 -1 0, limit lower=-2.6 upper=2.6 effort=18 velocity=40
- added joint rh_kfe: type revolute, parent rh_thigh, child rh_shank, origin xyz=0.0 -0.049 -0.2085 rpy=0.0 0 0.0, axis 0 -1 0, limit lower=-2.6 upper=2.6 effort=18 velocity=40
- added joint rh_shank_to_foot: type fixed, parent rh_shank, child rh_foot, origin xyz=0.0 0.0 -0.22 rpy=0.0 0.0 0.0
