Commit message: update knee joint limits on URDF, new URDF with rotor inertias (thanks Sehwan)

File: resources/robots/mini_cheetah/urdf/mini_cheetah_rotor.urdf (robot description, URDF)
Before this commit: robot mini_cheetah, 17 links, 16 joints
Links:
- link base: mass 3.3 -> 3.96
Joints:
- joint lh_kfe: limit lower=0.12 upper=4.97 effort=28 velocity=26.8 -> lower=-2.7 upper=2.7 effort=28 velocity=26.8
