Commit message: fix swing/stance rewards, zero-out avg_action on reset

File: resources/robots/mini_cheetah/urdf/mini_cheetah_simple.urdf (robot description, URDF)
Before this commit: robot mini_cheetah_vision, 17 links, 16 joints
Links:
- link lf_shank: geometry collision cylinder length=0.15 radius=0.01; visual mesh filename=meshes/lower_leg.dae
- link lh_hip: geometry collision cylinder length=0.01 radius=0.0475; visual mesh filename=meshes/mini_vision_abd.dae
- link lh_shank: geometry collision cylinder length=0.15 radius=0.01; visual mesh filename=meshes/lower_leg.dae
- link lh_thigh: geometry collision cylinder length=0.17 radius=0.015; visual mesh filename=meshes/mini_vision_upper_leg.dae
- link rf_hip: geometry collision cylinder length=0.01 radius=0.0475; visual mesh filename=meshes/mini_vision_abd.dae
- link rf_shank: geometry collision cylinder length=0.15 radius=0.01; visual mesh filename=meshes/lower_leg.dae
- link rf_thigh: geometry collision cylinder length=0.17 radius=0.015; visual mesh filename=meshes/mini_vision_upper_leg.dae
- link rh_hip: geometry collision cylinder length=0.01 radius=0.0475; visual mesh filename=meshes/mini_vision_abd.dae
- link rh_shank: geometry collision cylinder length=0.15 radius=0.01; visual mesh filename=meshes/lower_leg.dae
- link rh_thigh: geometry collision cylinder length=0.17 radius=0.015; visual mesh filename=meshes/mini_vision_upper_leg.dae

Commit message: small  changes for testing fixed `state_estimator` branch on rsl_rl

File: resources/robots/mini_cheetah/urdf/mini_cheetah_simple.urdf (robot description, URDF)
Before this commit: robot mini_cheetah_vision, 17 links, 16 joints
Links:
- link base: geometry collision box size=0.23 0.18 0.15; visual mesh filename=meshes/mini_vision_body.dae
- link lf_hip: geometry collision mesh filename=meshes/mini_vision_abd.dae; visual mesh filename=meshes/mini_vision_abd.dae
- link lf_shank: geometry collision mesh filename=meshes/lower_leg.dae; visual mesh filename=meshes/lower_leg.dae
- link lf_thigh: geometry collision mesh filename=meshes/mini_vision_upper_leg.dae; visual mesh filename=meshes/mini_vision_upper_leg.dae
- link lh_hip: geometry collision mesh filename=meshes/mini_vision_abd.dae; visual mesh filename=meshes/mini_vision_abd.dae
- link lh_shank: geometry collision mesh filename=meshes/lower_leg.dae; visual mesh filename=meshes/lower_leg.dae
- link lh_thigh: geometry collision mesh filename=meshes/mini_vision_upper_leg.dae; visual mesh filename=meshes/mini_vision_upper_leg.dae
- link rf_hip: geometry collision mesh filename=meshes/mini_vision_abd.dae; visual mesh filename=meshes/mini_vision_abd.dae
- link rf_shank: geometry collision mesh filename=meshes/lower_leg.dae; visual mesh filename=meshes/lower_leg.dae
- link rf_thigh: geometry collision mesh filename=meshes/mini_vision_upper_leg.dae; visual mesh filename=meshes/mini_vision_upper_leg.dae
- link rh_hip: geometry collision mesh filename=meshes/mini_vision_abd.dae; visual mesh filename=meshes/mini_vision_abd.dae
- link rh_shank: geometry collision mesh filename=meshes/lower_leg.dae; visual mesh filename=meshes/lower_leg.dae
- link rh_thigh: geometry collision mesh filename=meshes/mini_vision_upper_leg.dae; visual mesh filename=meshes/mini_vision_upper_leg.dae

Commit message: DECENT TUNED May19 Thursday

File: resources/robots/mini_cheetah/urdf/mini_cheetah_simple.urdf (robot description, URDF)
Before this commit: robot mini_cheetah, 17 links, 16 joints
Links:
- link base: geometry collision box size=0.23 0.18 0.2; visual mesh filename=meshes/mini_vision_body.dae

Commit message: added the new URDF for the mini cheetah (#22)
* added the new URDF for the mini cheetah

* made the paths of the URDFs in the matlab script relative

* [wip] did a simple collision for the MC for only one leg.

* fix mini_cheetah_simple urdf to use simple geometry for all collision boxes, have corrected torque and velocity limits. Tested with ref_SE_config

* match up limits etc. between  and

* remove . The shank collision box is approximated from the mesh and oversized, which always creates instant-collisions. Since the two URDFs cannot be made equivalent, better to avoid the possibility of training with the wrong one imho.

* use  for all configs

* adjust for Charles' code review

* removed unnecessary rotations of the shank, and shortened the shank to avoid false self-collisions and detecting overlap with the foot

* warning comment in matlab

Co-authored-by: Steve Heim <heim.steve@gmail.com>
Co-authored-by: Charles Khazoom <charles.khazoom@hotmail.com>

File: resources/robots/mini_cheetah/urdf/mini_cheetah_simple.urdf (robot description, URDF)
Before this commit: robot mini_cheetah, 17 links, 16 joints
Links:
- link base: geometry collision box size=0.30 0.20 0.10; visual mesh filename=meshes/mini_vision_body.dae
- link lf_foot: geometry collision sphere radius=0.0202
- link lf_hip: geometry visual mesh filename=meshes/mini_vision_abd.dae
- link lf_shank: geometry collision cylinder length=0.1 radius=0.01; visual mesh filename=meshes/lower_leg.dae
- link lf_thigh: geometry collision cylinder length=0.17 radius=0.015; visual mesh filename=meshes/mini_vision_upper_leg.dae
- link lh_foot: geometry collision sphere radius=0.0202
- link lh_hip: geometry visual mesh filename=meshes/mini_vision_abd.dae
- link lh_shank: geometry collision cylinder length=0.1 radius=0.01; visual mesh filename=meshes/lower_leg.dae
- link lh_thigh: geometry collision cylinder length=0.17 radius=0.015; visual mesh filename=meshes/mini_vision_upper_leg.dae
- link rf_foot: geometry collision sphere radius=0.0202
- link rf_hip: geometry visual mesh filename=meshes/mini_vision_abd.dae
- link rf_shank: geometry collision cylinder length=0.1 radius=0.01; visual mesh filename=meshes/lower_leg.dae
- link rf_thigh: geometry collision cylinder length=0.17 radius=0.015; visual mesh filename=meshes/mini_vision_upper_leg.dae
- link rh_foot: geometry collision sphere radius=0.0202
- link rh_hip: geometry visual mesh filename=meshes/mini_vision_abd.dae
- link rh_shank: geometry collision cylinder length=0.1 radius=0.01; visual mesh filename=meshes/lower_leg.dae
- link rh_thigh: geometry collision cylinder length=0.17 radius=0.015; visual mesh filename=meshes/mini_vision_upper_leg.dae
Joints:
- joint lf_haa: limit lower=-1.6 upper=1.6 effort=18 velocity=40 -> lower=-1.5 upper=1.5 effort=18 velocity=41
- joint lf_hfe: limit lower=-2.6 upper=2.6 effort=18 velocity=40 -> lower=-2.6 upper=2.6 effort=18 velocity=41
- joint lf_kfe: limit lower=-2.6 upper=2.6 effort=26 velocity=26 -> lower=0.12 upper=4.97 effort=28 velocity=26.8
- joint lh_haa: limit lower=-1.6 upper=1.6 effort=18 velocity=40 -> lower=-1.5 upper=1.5 effort=18 velocity=41
- joint lh_hfe: limit lower=-2.6 upper=2.6 effort=18 velocity=40 -> lower=-2.6 upper=2.6 effort=18 velocity=41
- joint lh_kfe: limit lower=-2.6 upper=2.6 effort=18 velocity=40 -> lower=0.12 upper=4.97 effort=28 velocity=26.8
- joint rf_haa: limit lower=-1.6 upper=1.6 effort=18 velocity=40 -> lower=-1.5 upper=1.5 effort=18 velocity=41
- joint rf_hfe: limit lower=-2.6 upper=2.6 effort=18 velocity=40 -> lower=-2.6 upper=2.6 effort=18 velocity=41
- joint rf_kfe: limit lower=-2.6 upper=2.6 effort=18 velocity=40 -> lower=0.12 upper=4.97 effort=28 velocity=26.8
- joint rh_haa: limit lower=-1.6 upper=1.6 effort=18 velocity=40 -> lower=-1.5 upper=1.5 effort=18 velocity=41
- joint rh_hfe: limit lower=-2.6 upper=2.6 effort=18 velocity=40 -> lower=-2.6 upper=2.6 effort=18 velocity=41
- joint rh_kfe: limit lower=-2.6 upper=2.6 effort=18 velocity=40 -> lower=0.12 upper=4.97 effort=28 velocity=26.8

Commit message: Mini Cheetah leg reordering to match Robot Software (#43)
* Update mini_cheetah_config.py

Update hip names in default joint angles

* Update ref_SE_config.py

Update hip names in default joint angles

* Legs reordered in URDF

Renamed legs to alphanumerically sort to same order as Robot Software

* flipping signs of right thigh link CoMs

* Update mini_cheetah_simple.urdf

* Update mini_cheetah_config.py

* Update ref_SE_config.py

* Abstract away dof_name enumeration from mc envs

* Update ref_SE_config.py

* Update mini_cheetah_config.py

* handle  only once per dof

Co-authored-by: saloutos <saloutos96@gmail.com>
Co-authored-by: Steve Heim <heim.steve@gmail.com>

File: resources/robots/mini_cheetah/urdf/mini_cheetah_simple.urdf (robot description, URDF)
Before this commit: robot mini_cheetah, 17 links, 16 joints
Joints:
- removed joint lf_haa
- removed joint lh_haa
- removed joint rf_haa
- removed joint rh_haa
- added joint 1_rf_haa: type revolute, parent base, child rf_hip, origin xyz=0.14775 -0.049 0.0 rpy=0 0 0, axis 1 0 0, limit lower=-1.5 upper=1.5 effort=18 velocity=41
- added joint 2_lf_haa: type revolute, parent base, child lf_hip, origin xyz=0.14775 0.049 0.0 rpy=0 0 0, axis 1 0 0, limit lower=-1.5 upper=1.5 effort=18 velocity=41
- added joint 3_rh_haa: type revolute, parent base, child rh_hip, origin xyz=-0.14775 -0.049 0.0 rpy=0 3.141592 0, axis -1 0 0, limit lower=-1.5 upper=1.5 effort=18 velocity=41
- added joint 4_lh_haa: type revolute, parent base, child lh_hip, origin xyz=-0.14775 0.049 0.0 rpy=0 3.141592 0, axis -1 0 0, limit lower=-1.5 upper=1.5 effort=18 velocity=41

Commit message: debugging legacy differences

File: resources/robots/mini_cheetah/urdf/mini_cheetah_simple.urdf (robot description, URDF)
Before this commit: robot mini_cheetah, 17 links, 16 joints
Joints:
- joint lh_kfe: limit lower=0.12 upper=4.97 effort=28 velocity=26.8 -> lower=-2.7 upper=2.7 effort=28 velocity=26.8
