Commit message: fixed base cartpole environment

File: resources/robots/cartpole/urdf/cartpole.urdf (robot description, URDF)
Before this commit: robot cartpole, 3 links, 2 joints
Joints:
- joint cart_to_pole: limit effort=1000.0 velocity=8 -> velocity=20
- joint slider_to_cart: limit lower=-4 upper=4 effort=1000.0 velocity=100 -> lower=-4 upper=4 effort=10.0 velocity=100

Commit message: 128 cartpole rewards not calculating correctly (#135)
* working training pipeline for cartpole to actually learn swing-up

* clean up play

* make cartpole physically slower (longer pole), some tuning. swings up, doesn't balance perfectly

* Tweak reward function and weights for more consistent balancing. Trains in approx 500-750 iterations

* working training pipeline for cartpole to actually learn swing-up

* clean up play

* make cartpole physically slower (longer pole), some tuning. swings up, doesn't balance perfectly

* Tweak reward function and weights for more consistent balancing. Trains in approx 500-750 iterations

* tweaked scalings, added a reward for energy pumping

---------

Co-authored-by: kendrick <ke26966@mit.edu>

File: resources/robots/cartpole/urdf/cartpole.urdf (robot description, URDF)
Before this commit: robot cartpole, 3 links, 2 joints
Links:
- link pole: geometry collision box size=0.04 0.06 2.0; visual box size=0.04 0.06 2.0
Joints:
- joint slider_to_cart: origin xyz=0 0 0 -> xyz=0 0 0.1
